File: PCB/DE10-lite_shield/_autosave-DE10-lite_shield.kicad_pcb (KiCad board)
At the start: 4 copper layers, 97.5 x 80 mm, 102 parts, among them J1 Conn_01x04, J10 Conn_01x02, J11 SM04B-SRSS-TB(LF)(SN), J12 SM04B-SRSS-TB(LF)(SN), J2 Conn_01x04, J3 Screw_Terminal_01x02, J4 USB4056-03-A, J5 Conn_01x05, J6 Conn_01x05, J7 Conn_01x05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

Commit message: PCB almost done
Parts:
- moved C15 101.6 mm to (149.3, 102.7)
- moved C13 76.9 mm to (181.4, 64.1), turned to 180 degrees
- moved C12 1.05 mm to (181.4, 65.2)
- moved U2 1.05 mm to (183.4, 68.9)
- moved R11 1.05 mm to (178.1, 67.0)
- moved R9 1.05 mm to (178.1, 68.2)
- moved R8 0.06 mm to (178.3, 75.3)
Routing:
- net EN: track 36.4 -> 80.9 mm
- net IO0: track 63.9 -> 102.3 mm
- net +3V3: track 16.8 -> 19.6 mm
- net GND: track 50.1 -> 52.9 mm
- net RTS: track 16.8 -> 15.7 mm
- net /USB_VBUS: track 4.79 -> 5.84 mm
- net /DP: track 12.9 -> 14.0 mm
- net /DN: track 13.3 -> 14.3 mm
- net DTR: track 21.7 -> 21.1 mm
- net I2C1_INT: track 34.7 -> 34.0 mm

Commit message: Changed configs
Parts:
- added C24: 10u, Capacitor_SMD:C_0402_1005Metric, F.Cu at (162.5, 127.9)
- moved C22 84.6 mm to (160.4, 127.9), turned to -90 degrees
- moved C21 83.8 mm to (161.4, 127.9), turned to -90 degrees
- moved C15 0.30 mm to (149.3, 102.4)
- moved C16 0.27 mm to (149.3, 97.2)
Routing:
- net +3V3: track 19.6 -> 23.0 mm
- net GND: track 52.9 -> 54.8 mm, vias 46 -> 45
