File: PCB/DE10-lite_shield/DE10-lite_shield.kicad_pcb (KiCad board)
At the start: 4 copper layers, 97.5 x 80 mm, 102 parts, among them J1 Conn_01x04, J10 Conn_01x02, J11 SM04B-SRSS-TB(LF)(SN), J12 SM04B-SRSS-TB(LF)(SN), J2 Conn_01x04, J3 Screw_Terminal_01x02, J4 USB4056-03-A, J5 Conn_01x05, J6 Conn_01x05, J7 Conn_01x05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

Commit message: FINISHED CIRCUIT BOARD IN 24 HOURS
Parts:
- removed JP7, JP8: Jumper_2_Open, Connector_PinHeader_2.54mm:PinHeader_1x02_P2.54mm_Vertical
- added C24: 10u, Capacitor_SMD:C_0402_1005Metric, F.Cu at (162.5, 127.9)
- added J10: Conn_01x02, Connector_PinHeader_2.54mm:PinHeader_1x02_P2.54mm_Vertical, F.Cu at (103.4, 122.0)
- added J10: Conn_01x02, Connector_PinHeader_2.54mm:PinHeader_1x02_P2.54mm_Vertical, F.Cu at (118.1, 114.9)
- added JP9: Jumper_3_Open, Connector_PinHeader_2.54mm:PinHeader_1x03_P2.54mm_Vertical, F.Cu at (160.1, 98.9)
- added REF**: ESD-Logo_6.6x6mm_SilkScreen, Symbol:ESD-Logo_6.6x6mm_SilkScreen, B.Cu at (169.8, 123.8)
- added REF**: KiCad-Logo2_5mm_SilkScreen, Symbol:KiCad-Logo2_5mm_SilkScreen, B.Cu at (183.0, 124.0)
- added REF**: WEEE-Logo_4.2x6mm_SilkScreen, Symbol:WEEE-Logo_4.2x6mm_SilkScreen, B.Cu at (161.3, 123.8)
- J9: moved to B.Cu
- SW1: footprint Connector_PinHeader_2.54mm:PinHeader_1x03_P2.54mm_Vertical -> footprints:Toggle_switch
- moved R25 131.4 mm to (128.8, 107.8), turned to 90 degrees
- moved R24 130.3 mm to (129.9, 107.8), turned to 90 degrees
- moved R15 111.6 mm to (135.1, 117.8)
- moved C15 99.8 mm to (151.1, 102.4)
- moved D5 97.9 mm to (164.2, 118.0), turned to 180 degrees
- moved R28 96.0 mm to (164.3, 119.5), turned to 180 degrees
- moved R26 95.9 mm to (164.3, 114.5), turned to 180 degrees
- moved R22 94.3 mm to (177.6, 64.9), turned to -90 degrees
- moved R21 93.3 mm to (178.6, 63.2), turned to -90 degrees
- moved D4 88.3 mm to (164.2, 116.0), turned to 180 degrees
- moved R20 87.2 mm to (174.3, 84.6), turned to -90 degrees
- moved R19 86.6 mm to (173.8, 86.2), turned to 180 degrees
- moved C22 84.6 mm to (160.4, 127.9), turned to -90 degrees
- moved C21 83.8 mm to (161.4, 127.9), turned to -90 degrees
- moved R23 79.6 mm to (185.5, 79.7)
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Connections:
- A2 pad 10: /MOTOR2_MS1 -> /MOTOR1_MS1
- A2 pad 11: /MOTOR2_MS2 -> /MOTOR1_MS2
- A2 pad 12: /MOTOR2_MS3 -> /MOTOR1_MS3
- A2 pad 13: /MOTOR2_RST -> /MOTOR1_RST
- A2 pad 14: /MOTOR2_RST -> /MOTOR1_RST
- A2 pad 15: MOTOR2_STEP_IN -> MOTOR1_STEP
- A2 pad 16: MOTOR2_DIR -> MOTOR1_DIR
- A2 pad 3: /MOTOR2_1B -> /MOTOR1_1B
- A2 pad 4: /MOTOR2_1A -> /MOTOR1_1A
- A2 pad 5: /MOTOR2_2A -> /MOTOR1_2A
- A2 pad 6: /MOTOR2_2B -> /MOTOR1_2B
- A3 pad 10: /MOTOR1_MS1 -> /MOTOR2_MS1
- A3 pad 11: /MOTOR1_MS2 -> /MOTOR2_MS2
- A3 pad 12: /MOTOR1_MS3 -> /MOTOR2_MS3
- A3 pad 13: /MOTOR1_RST -> /MOTOR2_RST
- A3 pad 14: /MOTOR1_RST -> /MOTOR2_RST
- A3 pad 15: MOTOR1_STEP -> MOTOR2_STEP_IN
- A3 pad 16: MOTOR1_DIR -> MOTOR2_DIR
- A3 pad 3: /MOTOR1_1B -> /MOTOR2_1B
- A3 pad 4: /MOTOR1_1A -> /MOTOR2_1A
- A3 pad 5: /MOTOR1_2A -> /MOTOR2_2A
- A3 pad 6: /MOTOR1_2B -> /MOTOR2_2B
- J1 pad 1: /MOTOR1_1B -> /MOTOR2_1B
- J1 pad 2: /MOTOR1_1A -> /MOTOR2_1A
- J1 pad 3: /MOTOR1_2A -> /MOTOR2_2A
- J1 pad 4: /MOTOR1_2B -> /MOTOR2_2B
- J11 pad S1: GND -> unconnected-(J11-SHIELD-PadS1)
- J11 pad S2: GND -> unconnected-(J11-SHIELD-PadS1)
- J12 pad S1: GND -> unconnected-(J12-SHIELD-PadS1)
- J12 pad S2: GND -> unconnected-(J12-SHIELD-PadS1)
- J2 pad 1: /MOTOR2_1B -> /MOTOR1_1B
- J2 pad 2: /MOTOR2_1A -> /MOTOR1_1A
- J2 pad 3: /MOTOR2_2A -> /MOTOR1_2A
- J2 pad 4: /MOTOR2_2B -> /MOTOR1_2B
- JP1 pad 2: /MOTOR1_MS1 -> /MOTOR2_MS1
- JP3 pad 2: /MOTOR1_MS3 -> /MOTOR2_MS3
- JP4 pad 2: /MOTOR2_MS1 -> /MOTOR1_MS1
- JP5 pad 2: /MOTOR2_MS2 -> /MOTOR1_MS2
- JP6 pad 2: /MOTOR2_MS3 -> /MOTOR1_MS3
- U1 pad 27: MOTOR2_DIR -> MOTOR1_DIR
- U1 pad 8: MOTOR1_DIR -> MOTOR2_DIR
- locked pad 2: /MOTOR1_MS2 -> /MOTOR2_MS2
Routing:
- net MOTOR1_STEP: track 9.46 -> 93.1 mm, vias 1 -> 2
- net SCL0: track 0.00 -> 79.3 mm
- net SDA0: track 0.00 -> 77.6 mm, vias 0 -> 1
- net VBUS/2: track 0.00 -> 75.3 mm, vias 0 -> 4
- net /FPGA_LED_A: track 0.00 -> 73.9 mm, vias 0 -> 1
- net SCL1: track 0.00 -> 73.0 mm
- net SDA1: track 0.00 -> 71.3 mm
- net FPGA_INT: track 0.00 -> 68.5 mm, vias 0 -> 1
- net MOTOR1_DIR: track 11.1 -> 77.6 mm, vias 0 -> 1
- net +3V3: track 16.8 -> 83.0 mm, vias 1 -> 117
- net FPGA_GPIO: track 0.00 -> 65.3 mm, vias 0 -> 1
- net BATT/4: track 0.00 -> 53.5 mm, vias 0 -> 2
- net EN: track 36.4 -> 81.7 mm
- net IO0: track 63.9 -> 108.4 mm
- net MOTOR2_DIR: track 29.6 -> 55.8 mm
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- added copper zone on B.Cu, net +3V3
- added copper zone on F.Cu, net +3V3
- added copper zone on B.Cu, net /VIN_FUSED
Other:
- board text added: "+"
- board text added: "+5V"
- board text added: "-"
- board text added: "10V MAX INPUT"
- board text added: "3V3"
- board text added: "5V0"
- board text added: "BOOT"
- board text added: "DE10-Lite Shield V1"
- board text added: "Designed by Ben Smith 2023"
- board text added: "EN"
- board text added: "ESP32"
- board text added: "ESP32 LED"
- board text added: "FPGA LED"
- board text added: "FUSE"
- board text added: "GND"
- board text added: "GROUP 1"
- board text added: "I2C0"
- board text added: "I2C1"
- board text added: "I2C2"
- board text added: "I2C3"
- board text added: "I2C4"
- board text added: "I2C5"
- board text added: "IMU"
- board text added: "INT"
- board text added: "Left for shared STEP pin Right for individual STEP pins"
- board text added: "MOTOR1"
- board text added: "MOTOR2"
- board text added: "MS1"
- board text added: "MS2"
- board text added: "MS3"
- board text added: "OFF"
- board text added: "ON"
- board text added: "S"
- board text added: "SCL"
- board text added: "SDA"
- board text added: "SERVO"

Commit message: Finished PCB
Parts:
- J9: moved to F.Cu
- turned J9 to 90 degrees
Connections:
- U4 pad 25: unconnected-(U4-1EP-Pad25) -> GND

Commit message: Fixed unrouted nets
Routing:
- net +BATT: track 1.50 -> 12.8 mm, vias 2 -> 3
- net +1V8: track 29.6 -> 36.5 mm, vias 0 -> 2
- net +3V3: track 83.0 -> 88.9 mm
